File: pcb/climatedisplay.kicad_sch (KiCad schematic)
At the start: 27 parts, among them J1 Serial, J2 USB-C 6-Pin, SW1 RESET, SW2 FLASH, U1 ESP-12F, U2 74AHCT1G08, U3 74AHCT1G08, U4 74AHCT1G08, U5 AMS1117-3.3

Commit message: fix: footprints U2-U4
Parts:
- U2, U3, U4: footprint Package_TO_SOT_SMD:SOT-23-5 -> Package_TO_SOT_SMD:SOT-353_SC-70-5
Changed lines of the file:
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@@
 			)
 		)
-		(property "Footprint" "Package_TO_SOT_SMD:SOT-23-5"
+		(property "Footprint" "Package_TO_SOT_SMD:SOT-353_SC-70-5"
 			(at 232.41 95.25 0)
 			(effects
@@
 			)
 		)
-		(property "Footprint" "Package_TO_SOT_SMD:SOT-23-5"
+		(property "Footprint" "Package_TO_SOT_SMD:SOT-353_SC-70-5"
 			(at 207.01 123.19 0)
 			(effects
@@
 			)
 		)
-		(property "Footprint" "Package_TO_SOT_SMD:SOT-23-5"
+		(property "Footprint" "Package_TO_SOT_SMD:SOT-353_SC-70-5"
 			(at 175.26 95.25 0)
 			(effects
